File: Hardware/BatteryCharger/BatteryCharger.kicad_sch (KiCad schematic)
At the start: 15 parts, among them Q1 TIP32C

Commit message: Progress Check-in, working on schematic
Parts:
- added R10: DNF, Resistor_THT:R_Axial_DIN0207_L6.3mm_D2.5mm_P10.16mm_Horizontal, symbol Device:R_Small
- added R8: 10k0, Resistor_THT:R_Axial_DIN0207_L6.3mm_D2.5mm_P10.16mm_Horizontal, symbol Device:R_Small
- C3: renamed from C1; value C_Small -> 01uF
Connections:
- net GND: now also R10.2
- net Out: now reaches D1.1 (K), R3.1, R4.1
- net Out: now also R8.2
- net at R11.2, R12.2, R9.2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: now also R10.1
- net In: now reaches R1.1, U1.3 (ISNSP), U1.5 (IN)
- net at U1.9 (STAT2): now also R8.1
Changed lines of the file:
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@@
+	)
+	(junction
+		(at 194.31 93.98)
+		(diameter 0)
+		(color 0 0 0 0)
 	)
 	(junction
@@
 	)
 	(junction
+		(at 194.31 36.83)
+		(diameter 0)
+		(color 0 0 0 0)
+	)
+	(junction
 		(at 194.31 72.39)
 		(diameter 0)
@@
 	(wire
 		(pts
+			(xy 208.28 36.83) (xy 194.31 36.83)
+		)
+		(stroke
+			(width 0)
+			(type default)
+		)
+	)
+	(wire
+		(pts
 			(xy 146.05 36.83) (xy 146.05 45.72)
 		)
@@
 	(wire
 		(pts
+			(xy 180.34 99.06) (xy 185.42 99.06)
+		)
+		(stroke
+			(width 0)
+			(type default)
+		)
+	)
+	(wire
+		(pts
 			(xy 139.7 67.31) (xy 120.65 67.31)
 		)
@@
 	(wire
 		(pts
+			(xy 194.31 107.95) (xy 194.31 114.3)
+		)
+		(stroke
+			(width 0)
+			(type default)
+		)
+	)
+	(wire
+		(pts
 			(xy 127 76.2) (xy 120.65 76.2)
 		)
@@
 	(wire
 		(pts
+			(xy 194.31 93.98) (xy 194.31 102.87)
+		)
+		(stroke
+			(width 0)
+			(type default)
+		)
+	)
+	(wire
+		(pts
 			(xy 194.31 93.98) (xy 194.31 88.9)
 		)
@@
 	(wire
 		(pts
+			(xy 190.5 99.06) (xy 208.28 99.06)
+		)
+		(stroke
+			(width 0)
+			(type default)
+		)
+	)
+	(wire
+		(pts
 			(xy 146.05 57.15) (xy 146.05 45.72)
 		)
@@
 			(width 0)
 			(type default)
+		)
+	)
+	(wire
+		(pts
+			(xy 208.28 99.06) (xy 208.28 36.83)
+		)
+		(stroke
+			(width 0)
+			(type default)
+		)
+	)
+	(label "In"
+		(at 102.87 36.83 0)
+		(fields_autoplaced yes)
+		(effects
+			(font
+				(size 1.27 1.27)
+			)
+			(justify left bottom)
+		)
+	)
+	(label "Out"
+		(at 190.5 36.83 0)
+		(fields_autoplaced yes)
+		(effects
+			(font
+				(size 1.27 1.27)
+			)
+			(justify left bottom)
 		)
 	)
@@
 	(symbol
 		(lib_id "Device:R_Small")
+		(at 194.31 105.41 0)
+		(unit 1)
+		(exclude_from_sim no)
+		(in_bom yes)
+		(on_board yes)
+		(dnp no)
+		(property "Reference" "R10"
+			(at 191.262 104.648 0)
+			(effects
+				(font
+					(size 1.27 1.27)
+				)
+			)
+		)
+		(property "Value" "DNF"
+			(at 191.262 106.68 0)
+			(effects
+				(font
+					(size 1.27 1.27)
+				)
+			)
+		)
+		(property "Footprint" "Resistor_THT:R_Axial_DIN0207_L6.3mm_D2.5mm_P10.16mm_Horizontal"
+			(at 194.31 105.41 0)
+			(effects
+				(font
+					(size 1.27 1.27)
+				)
+				(hide yes)
+			)
+		)
+		(property "Datasheet" "~"
+			(at 194.31 105.41 0)
+			(effects
+				(font
+					(size 1.27 1.27)
+				)
+				(hide yes)
+			)
+		)
+		(property "Description" ""
+			(at 194.31 105.41 0)
+			(effects
+				(font
+					(size 1.27 1.27)
+				)
+				(hide yes)
+			)
+		)
+		(pin "1"
+		)
+		(pin "2"
+		)
+		(instances
+			(project "BatteryCharger"
+				(path "/513cbfc7-d5e1-4614-b530-d0a3d04d78fb"
+					(reference "R10")
+					(unit 1)
+				)
+			)
+		)
+	)
+	(symbol
+		(lib_id "Device:R_Small")
 		(at 187.96 88.9 90)
 		(unit 1)
@@
 	)
 	(symbol
+		(lib_id "Device:R_Small")
+		(at 187.96 99.06 90)
+		(unit 1)
+		(exclude_from_sim no)
+		(in_bom yes)
+		(on_board yes)
+		(dnp no)
+		(property "Reference" "R8"
+			(at 184.912 97.028 90)
+			(effects
+				(font
+					(size 1.27 1.27)
+				)
+			)
+		)
+		(property "Value" "10k0"
+			(at 190.246 97.028 90)
+			(effects
+				(font
+					(size 1.27 1.27)
+				)
+			)
+		)
+		(property "Footprint" "Resistor_THT:R_Axial_DIN0207_L6.3mm_D2.5mm_P10.16mm_Horizontal"
+			(at 187.96 99.06 0)
+			(effects
+				(font
+					(size 1.27 1.27)
+				)
+				(hide yes)
+			)
+		)
+		(property "Datasheet" "~"
+			(at 187.96 99.06 0)
+			(effects
+				(font
+					(size 1.27 1.27)
+				)
+				(hide yes)
+			)
+		)
+		(property "Description" ""
+			(at 187.96 99.06 0)
+			(effects
+				(font
+					(size 1.27 1.27)
+				)
+				(hide yes)
+			)
+		)
+		(pin "1"
+		)
+		(pin "2"
+		)
+		(instances
+			(project "BatteryCharger"
+				(path "/513cbfc7-d5e1-4614-b530-d0a3d04d78fb"
+					(reference "R8")
+					(unit 1)
+				)
+			)
+		)
+	)
+	(symbol
 		(lib_id "MyParts:BQ24450")
 		(at 144.78 63.5 0)
@@
 		(dnp no)
 		(fields_autoplaced yes)
-		(property "Reference" "C1"
-			(at 162.3441 109.2842 0)
+		(property "Reference" "C3"
+			(at 162.56 109.2262 0)
 			(effects
 				(font
@@
 			)
 		)
-		(property "Value" "C_Small"
-			(at 162.3441 111.7084 0)
+		(property "Value" "01uF"
+			(at 162.56 111.7662 0)
 			(effects
 				(font
@@
 			(project "BatteryCharger"
 				(path "/513cbfc7-d5e1-4614-b530-d0a3d04d78fb"
-					(reference "C1")
+					(reference "C3")
 					(unit 1)
 				)
@@
 	(symbol
 		(lib_id "power:GND")
-		(at 203.2 101.6 0)
+		(at 194.31 114.3 0)
 		(unit 1)
 		(exclude_from_sim no)
@@
 		(fields_autoplaced yes)
 		(property "Reference" "#PWR03"
-			(at 203.2 107.95 0)
+			(at 194.31 120.65 0)
 			(effects
 				(font
@@
 		)
 		(property "Value" "GND"
-			(at 203.2 105.7331 0)
+			(at 194.31 118.4331 0)
 			(effects
 				(font
@@
 		)
 		(property "Footprint" ""
-			(at 203.2 101.6 0)
+			(at 194.31 114.3 0)
 			(effects
 				(font
@@
 		)
 		(property "Datasheet" ""
-			(at 203.2 101.6 0)
+			(at 194.31 114.3 0)
 			(effects
 				(font
@@
 		)
 		(property "Description" ""
-			(at 203.2 101.6 0)
-			(effects
-				(font
+			(at 194.31 114.3 0)
+			(effects
+				(font

Commit message: Progress check-in: working on charger schematic
Parts:
- added C4: DNF, Capacitor_THT:C_Axial_L5.1mm_D3.1mm_P10.00mm_Horizontal, symbol Device:C_Small
- added J1, J2: Screw_Terminal_01x02, symbol Connector:Screw_Terminal_01x02
- C3: footprint (none) -> Capacitor_THT:C_Axial_L5.1mm_D3.1mm_P10.00mm_Horizontal
- JP1, JP2, JP3: footprint (none) -> Jumper:SolderJumper-3_P1.3mm_Bridged12_Pad1.0x1.5mm
- R1: footprint Diode_SMD:D_2512_6332Metric_Pad1.52x3.35mm_HandSolder -> MyParts:R_2512 Large Pad
- R2: footprint Diode_SMD:D_2512_6332Metric_Pad1.52x3.35mm_HandSolder -> Resistor_THT:R_Axial_DIN0207_L6.3mm_D2.5mm_P10.16mm_Horizontal
Connections:
- net GND: now also C4.2, J1.2 (Pin_2), J2.2 (Pin_2)
- net In: now also J1.1 (Pin_1)
- net Out: now also J2.1 (Pin_1)
- net at U1.1 (ISNS), U1.8 (BSTOP): now also C4.1

Commit message: Progress: Finished schematic, starting on PCB
Parts:
- J1, J2: value Screw_Terminal_01x02 -> Wurth 691313510002; footprint (none) -> MyParts-Mouser:Wurth_691313510002_Pluggable_Terminal_Block
Other:
- moved on the sheet: J2
Changed lines of the file:
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@@
 	(wire
 		(pts
-			(xy 212.09 39.37) (xy 212.09 43.18)
+			(xy 218.44 39.37) (xy 218.44 43.18)
 		)
 		(stroke
@@
 	(wire
 		(pts
-			(xy 208.28 36.83) (xy 212.09 36.83)
+			(xy 208.28 36.83) (xy 218.44 36.83)
 		)
 		(stroke
@@
 	(symbol
 		(lib_id "power:GND")
-		(at 212.09 43.18 0)
+		(at 218.44 43.18 0)
 		(unit 1)
 		(exclude_from_sim no)
@@
 		(fields_autoplaced yes)
 		(property "Reference" "#PWR06"
-			(at 212.09 49.53 0)
+			(at 218.44 49.53 0)
 			(effects
 				(font
@@
 		)
 		(property "Value" "GND"
-			(at 212.09 47.3131 0)
+			(at 218.44 47.3131 0)
 			(effects
 				(font
@@
 		)
 		(property "Footprint" ""
-			(at 212.09 43.18 0)
+			(at 218.44 43.18 0)
 			(effects
 				(font
@@
 		)
 		(property "Datasheet" ""
-			(at 212.09 43.18 0)
+			(at 218.44 43.18 0)
 			(effects
 				(font
@@
 		)
 		(property "Description" ""
-			(at 212.09 43.18 0)
+			(at 218.44 43.18 0)
 			(effects
 				(font
@@
 			)
 		)
-		(property "Value" "Screw_Terminal_01x02"
+		(property "Value" "Wurth 691313510002"
 			(at 95.25 39.3699 0)
 			(effects
@@
 			)
 		)
-		(property "Footprint" ""
+		(property "Footprint" "MyParts-Mouser:Wurth_691313510002_Pluggable_Terminal_Block"
 			(at 97.79 36.83 0)
 			(effects
@@
 	(symbol
 		(lib_id "Connector:Screw_Terminal_01x02")
-		(at 217.17 36.83 0)
+		(at 223.52 36.83 0)
 		(unit 1)
 		(exclude_from_sim no)
@@
 		(fields_autoplaced yes)
 		(property "Reference" "J2"
-			(at 219.71 36.8299 0)
+			(at 226.06 36.8299 0)
 			(effects
 				(font
@@
 			)
 		)
-		(property "Value" "Screw_Terminal_01x02"
-			(at 219.71 39.3699 0)
+		(property "Value" "Wurth 691313510002"
+			(at 226.06 39.3699 0)
 			(effects
 				(font
@@
 			)
 		)
-		(property "Footprint" ""
-			(at 217.17 36.83 0)
+		(property "Footprint" "MyParts-Mouser:Wurth_691313510002_Pluggable_Terminal_Block"
+			(at 223.52 36.83 0)
 			(effects
 				(font
@@
 		)
 		(property "Datasheet" "~"
-			(at 217.17 36.83 0)
+			(at 223.52 36.83 0)
 			(effects
 				(font
@@
 		)
 		(property "Description" "Generic screw terminal, single row, 01x02, script generated (kicad-library-utils/schlib/autogen/connector/)"
-			(at 217.17 36.83 0)
-			(effects
-				(font
+			(at 223.52 36.83 0)
+			(effects
+				(font

Commit message: Progress - Laying out PCB
Parts:
- C3: value 01uF -> 0u1F
Changed lines of the file:
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@@
 			)
 		)
-		(property "Value" "01uF"
+		(property "Value" "0u1F"
 			(at 162.56 111.7662 0)
 			(effects

Commit message: Fix error on charger PCB and add mounting holes to schematic
Parts:
- removed Q1: TIP32C, Package_TO_SOT_THT:TO-220-3_Vertical, symbol Simulation_SPICE:PNP
- added H1, H2, H3, H4: MountingHole, MyParts:MountingHole_3.2mm_M3, symbol Mechanical:MountingHole
- added Q1: TIP32C, Package_TO_SOT_THT:TO-220-3_Vertical, symbol Device:Q_PNP_BCE
Connections:
- net at D1.2 (A), JP2.3 (B): now also Q1.2 (C)
- net at U1.16 (DRVC): now also Q1.1 (B)
- net at JP1.3 (B), JP3.3 (B), R2.2: now also Q1.3 (E)
Other:
- note added: "Note: DNF = Do Not Fit"
