File: Hardware/AlarmUnit/AlarmUnit.kicad_sch (KiCad schematic)
At the start: 34 parts, among them J1 Screw_Terminal_01x08, J2 Screw_Terminal_01x08, J3 Screw_Terminal_01x08, J4 Screw_Terminal_01x02, J5 Screw_Terminal_01x02, J6 IDC_10 on CPU, J7 IDC_10 on IO board, Q1 2N7000, Q2 2N7000, Q3 P36NF06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

Commit message: Update schematic with CPU pins to connectors
Connections:
- net In_1_Buffered: now also J6.10 (Pin_10), J7.10 (Pin_10)
- net In_2_Buffered: now also J6.9 (Pin_9), J7.9 (Pin_9)
- net In_3_Buffered: now also J6.7 (Pin_7), J7.7 (Pin_7)
- net In_4_Buffered: now also J6.8 (Pin_8), J7.8 (Pin_8)
- net In_5_Buffered: now also J6.5 (Pin_5), J7.5 (Pin_5)
- net In_6_Buffered: now also J6.6 (Pin_6), J7.6 (Pin_6)
Changed lines of the file:
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@@
+		)
+	)
+	(label "In_5_Buffered"
+		(at 130.81 137.16 180)
+		(fields_autoplaced yes)
+		(effects
+			(font
+				(size 1.27 1.27)
+			)
+			(justify right bottom)
 		)
 	)
@@
 		)
 	)
+	(label "In_4_Buffered"
+		(at 143.51 139.7 0)
+		(fields_autoplaced yes)
+		(effects
+			(font
+				(size 1.27 1.27)
+			)
+			(justify left bottom)
+		)
+	)
 	(label "Input_1"
 		(at 210.82 24.13 0)
@@
 		)
 	)
+	(label "In_6_Buffered"
+		(at 143.51 137.16 0)
+		(fields_autoplaced yes)
+		(effects
+			(font
+				(size 1.27 1.27)
+			)
+			(justify left bottom)
+		)
+	)
 	(label "Input_Common"
 		(at 259.08 95.25 180)
@@
 		)
 	)
+	(label "In_3_Buffered"
+		(at 130.81 165.1 180)
+		(fields_autoplaced yes)
+		(effects
+			(font
+				(size 1.27 1.27)
+			)
+			(justify right bottom)
+		)
+	)
 	(label "Input_Common"
 		(at 259.08 46.99 180)
@@
 	)
 	(label "In_6_Buffered"
+		(at 143.51 162.56 0)
+		(fields_autoplaced yes)
+		(effects
+			(font
+				(size 1.27 1.27)
+			)
+			(justify left bottom)
+		)
+	)
+	(label "In_6_Buffered"
 		(at 113.03 82.55 180)
 		(fields_autoplaced yes)
@@
 		)
 	)
+	(label "In_4_Buffered"
+		(at 143.51 165.1 0)
+		(fields_autoplaced yes)
+		(effects
+			(font
+				(size 1.27 1.27)
+			)
+			(justify left bottom)
+		)
+	)
 	(label "Out_1_Buffered"
 		(at 163.83 72.39 0)
@@
 		)
 	)
+	(label "In_1_Buffered"
+		(at 143.51 142.24 0)
+		(fields_autoplaced yes)
+		(effects
+			(font
+				(size 1.27 1.27)
+			)
+			(justify left bottom)
+		)
+	)
+	(label "In_1_Buffered"
+		(at 143.51 167.64 0)
+		(fields_autoplaced yes)
+		(effects
+			(font
+				(size 1.27 1.27)
+			)
+			(justify left bottom)
+		)
+	)
 	(label "Out_2_Buffered"
 		(at 161.29 146.05 180)
@@
 		)
 	)
+	(label "In_2_Buffered"
+		(at 130.81 142.24 180)
+		(fields_autoplaced yes)
+		(effects
+			(font
+				(size 1.27 1.27)
+			)
+			(justify right bottom)
+		)
+	)
 	(label "Input_2"
 		(at 259.08 31.75 180)
@@
 		)
 	)
+	(label "In_3_Buffered"
+		(at 130.81 139.7 180)
+		(fields_autoplaced yes)
+		(effects
+			(font
+				(size 1.27 1.27)
+			)
+			(justify right bottom)
+		)
+	)
 	(label "In_2_Buffered"
 		(at 184.15 30.48 180)
@@
 		)
 	)
+	(label "In_5_Buffered"
+		(at 130.81 162.56 180)
+		(fields_autoplaced yes)
+		(effects
+			(font
+				(size 1.27 1.27)
+			)
+			(justify right bottom)
+		)
+	)
 	(label "In_1_Buffered"
 		(at 184.15 19.05 180)
@@
 		(fields_autoplaced yes)
 		(effects
+			(font
+				(size 1.27 1.27)
+			)
+			(justify right bottom)
+		)
+	)
+	(label "In_2_Buffered"
+		(at 130.81 167.64 180)
+		(fields_autoplaced yes)
+		(effects
